Commit message: sfbot 수정
링크의 이름을 겹치지 않도록 하였고, 접합 방식을 알맞게 수정함(회전)

File: sfbot/sfbot.urdf (robot description, URDF)
Before this commit: robot sfbot, 13 links, 14 joints
Links:
- removed link ak70-10-v1
- removed link 구성요소8
- added link ak70-10-v1_1, mass 2.1429063401431327; collision mesh filename=meshes/ak70-10-v1_1.stl scale=0.001 0.001 0.001; visual mesh filename=meshes/ak70-10-v1_1.stl scale=0.001 0.001 0.001
- added link ak70-10-v1_2, mass 2.1429063401431327; collision mesh filename=meshes/ak70-10-v1_2.stl scale=0.001 0.001 0.001; visual mesh filename=meshes/ak70-10-v1_2.stl scale=0.001 0.001 0.001
- added link 구성요소8_1, mass 0.668762166036501; collision mesh filename=meshes/구성요소8_1.stl scale=0.001 0.001 0.001; visual mesh filename=meshes/구성요소8_1.stl scale=0.001 0.001 0.001
- added link 구성요소8_2, mass 0.668762166036501; collision mesh filename=meshes/구성요소8_2.stl scale=0.001 0.001 0.001; visual mesh filename=meshes/구성요소8_2.stl scale=0.001 0.001 0.001
Joints:
- removed joint ak60-6v1-1-v1_강체-1
- removed joint ak70-10-v1_강체-10
- removed joint ak70-10-v1_강체-5
- removed joint ak70-10-v1_강체-9
- removed joint 구성요소6_강체-3
- removed joint 구성요소8_강체-17
- added joint ak60-6v1-1-v1_회전-1: type continuous, parent ak60-6v1-1-v1, child 구성요소11, origin xyz=0.0019298499999999997 -0.003603870000000001 0.02871041000000002 rpy=3.141592653589793 -1.5707963267948966 0, axis -0.990014 -0.12427100000000012 -0.066546
- added joint ak70-10-v1_1_회전-5: type continuous, parent ak70-10-v1_1, child 구성요소2, origin xyz=0.0 0.0 0.03905 rpy=-3.141592653589793 -1.5707963267948966 0, axis -1.0 -0.0 -7.888609052210118e-31
- added joint ak70-10-v1_2_강체-10: type fixed, parent ak70-10-v1_2, child 구성요소6, origin xyz=-0.02878305 0.0 -0.015413110000000004 rpy=1.5707963267948968 -0.0 -1.5707963267948966
- added joint ak70-10-v1_2_회전-9: type continuous, parent ak70-10-v1_2, child 구성요소5, origin xyz=0.005641909999999999 0.0 0.0030212099999999977 rpy=-1.5707963267948966 -0.0 -1.5707963267948966, axis -7.447951350553661e-31 0.47207000000000005 -0.881561
- added joint 구성요소8_1_강체-17: type fixed, parent 구성요소8_1, child 구성요소9, origin xyz=-0.009227670000000004 -0.07514998000000002 0.00028544999999999824 rpy=-3.141592653589793 5.8689517296745976e-18 2.775557561562892e-17
- added joint 구성요소9_강체-19: type fixed, parent 구성요소9, child 구성요소8_2, origin xyz=-0.07405115000000001 -3.552713678800501e-17 0.03965385000000001 rpy=-2.71281853479291e-18 5.651269022745248e-17 2.775557561562892e-17
- joint ak60-6v1-1-v1_강체-13: origin xyz=-4.338734978715565e-32 0.0 0.0275 rpy=3.141592653589793 -1.5707963267948966 0 -> xyz=0.0018300300000000003 -0.0034174600000000024 0.027225390000000012 rpy=3.141592653589793 -1.5707963267948966 0
- joint base_link_강체-4: child ak70-10-v1 -> ak70-10-v1_1
- joint 구성요소2_강체-6: origin xyz=0.02 0.0 1.5777218104420236e-32 rpy=-3.141592653589793 -1.5707963267948966 0 -> xyz=0.02 0.0 1.5777218104420236e-32 rpy=3.141592653589793 -1.5707963267948966 0
- joint 구성요소3_강체-7: origin xyz=0.015 0.02598076 0.01800000000000001 rpy=3.141592653589793 -0.0 0.0 -> xyz=-0.02998468 0.00095869 0.01800000000000001 rpy=-3.141592653589793 -3.944304526105059e-31 9.800333363043902e-30
- joint 구성요소4_강체-8: child ak70-10-v1 -> ak70-10-v1_2; origin xyz=-0.015 0.04225576 -0.056999999999999995 rpy=1.5707963267948966 -0.0 0.0 -> xyz=0.04433209 -0.00672424 -0.056999999999999995 rpy=1.5707963267948966 -7.888609052210118e-31 5.551115123118146e-17
- joint 구성요소5_강체-11: origin xyz=0.03249999999999998 0.024999999999999994 2.2114182278129884e-49 rpy=1.5707963267948966 -1.5707963267948966 0 -> xyz=0.03217546 -0.00776292 0.02420179 rpy=1.5707963267948966 -1.5707963267948966 0
- joint 구성요소7_강체-12: child 구성요소8 -> 구성요소8_1; origin xyz=1.0274702246948889e-140 0.0125 -0.01 rpy=0.0 -0.0 0.0 -> xyz=0.007983789999999998 0.012375179999999979 0.006274090000000001 rpy=-1.385805059804159e-19 -5.355483398803478e-17 2.7755575615628907e-17
- joint 구성요소9_강체-16: origin xyz=-0.015155440000000022 0.007250000000000014 -0.042 rpy=-1.5707963267948966 1.9721522630525295e-31 0.0 -> xyz=-0.029460129999999998 0.005041179999999947 0.033954930000000015 rpy=-1.5707963267948966 5.651269022745248e-17 2.775557561562892e-17

Commit message: Kor2Eng of Component name

File: sfbot/sfbot.urdf (robot description, URDF)
Before this commit: robot sfbot, 15 links, 14 joints
Links:
- removed link 구성요소10
- removed link 구성요소11
- removed link 구성요소2
- removed link 구성요소3
- removed link 구성요소4
- removed link 구성요소5
- removed link 구성요소6
- removed link 구성요소7
- removed link 구성요소8_1
- removed link 구성요소8_2
- removed link 구성요소9
- added link Component10, mass 0.13156890942165747; collision mesh filename=meshes/Component10.stl scale=0.001 0.001 0.001; visual mesh filename=meshes/Component10.stl scale=0.001 0.001 0.001
- added link Component11, mass 0.3456856671384452; collision mesh filename=meshes/Component11.stl scale=0.001 0.001 0.001; visual mesh filename=meshes/Component11.stl scale=0.001 0.001 0.001
- added link Component2, mass 1.0016922735671667; collision mesh filename=meshes/Component2.stl scale=0.001 0.001 0.001; visual mesh filename=meshes/Component2.stl scale=0.001 0.001 0.001
- added link Component3, mass 0.8807950300955173; collision mesh filename=meshes/Component3.stl scale=0.001 0.001 0.001; visual mesh filename=meshes/Component3.stl scale=0.001 0.001 0.001
- added link Component4, mass 0.6184682868789885; collision mesh filename=meshes/Component4.stl scale=0.001 0.001 0.001; visual mesh filename=meshes/Component4.stl scale=0.001 0.001 0.001
- added link Component5, mass 0.6082106863628858; collision mesh filename=meshes/Component5.stl scale=0.001 0.001 0.001; visual mesh filename=meshes/Component5.stl scale=0.001 0.001 0.001
- added link Component6, mass 0.8292297988354185; collision mesh filename=meshes/Component6.stl scale=0.001 0.001 0.001; visual mesh filename=meshes/Component6.stl scale=0.001 0.001 0.001
- added link Component7, mass 0.3722794963916967; collision mesh filename=meshes/Component7.stl scale=0.001 0.001 0.001; visual mesh filename=meshes/Component7.stl scale=0.001 0.001 0.001
- added link Component8_1, mass 0.668762166036501; collision mesh filename=meshes/Component8_1.stl scale=0.001 0.001 0.001; visual mesh filename=meshes/Component8_1.stl scale=0.001 0.001 0.001
- added link Component8_2, mass 0.668762166036501; collision mesh filename=meshes/Component8_2.stl scale=0.001 0.001 0.001; visual mesh filename=meshes/Component8_2.stl scale=0.001 0.001 0.001
- added link Component9, mass 0.6867109263567744; collision mesh filename=meshes/Component9.stl scale=0.001 0.001 0.001; visual mesh filename=meshes/Component9.stl scale=0.001 0.001 0.001
Joints:
- removed joint 구성요소2_강체-6
- removed joint 구성요소3_강체-7
- removed joint 구성요소4_강체-8
- removed joint 구성요소5_강체-11
- removed joint 구성요소7_강체-12
- removed joint 구성요소8_1_강체-17
- removed joint 구성요소9_강체-16
- removed joint 구성요소9_강체-19
- added joint Component2_강체-6: type fixed, parent Component2, child Component3, origin xyz=0.02 0.0 1.5777218104420236e-32 rpy=-3.141592653589793 -1.5707963267948966 0
- added joint Component3_강체-7: type fixed, parent Component3, child Component4, origin xyz=-0.0138827 -0.02659456 0.01800000000000001 rpy=3.141592653589793 -0.0 -1.6001510861891693e-31
- added joint Component4_강체-8: type fixed, parent Component4, child ak70-10-v1_2, origin xyz=0.01319128 -0.042854869999999996 -0.056999999999999995 rpy=1.5707963267948966 -0.0 3.2178910748521876e-30
- added joint Component5_강체-11: type fixed, parent Component5, child Component7, origin xyz=0.03168701 -0.024670539999999998 -0.00827939 rpy=1.5707963267948966 -1.5707963267948966 0
- added joint Component7_강체-12: type fixed, parent Component7, child Component8_1, origin xyz=0.002351049999999999 0.012187310000000019 0.010109000000000003 rpy=-7.227596320303442e-19 -6.261554580234533e-18 0.0
- added joint Component8_1_강체-17: type fixed, parent Component8_1, child Component9, origin xyz=-0.03080084 -0.06853650000000001 -0.009316940000000003 rpy=3.141592653589793 1.700735212931283e-18 -2.7755575615628914e-17
- added joint Component9_강체-16: type fixed, parent Component9, child ak60-6v1-1-v1, origin xyz=0.014937280000000018 0.010437270000000005 0.041402789999999995 rpy=-1.5707963267948966 -2.1956751568497123e-18 2.775557561562892e-17
- added joint Component9_강체-19: type fixed, parent Component9, child Component8_2, origin xyz=0.003568610000000043 0.0 0.08392416000000001 rpy=2.3777449427013474e-18 -2.1956751568497123e-18 2.775557561562892e-17
- joint ak60-6v1-1-v1_강체-13: child 구성요소10 -> Component10; origin xyz=0.0018300300000000003 -0.0034174600000000024 0.027225390000000012 rpy=3.141592653589793 -1.5707963267948966 0 -> xyz=-0.0061069500000000025 -0.000259680000000001 0.02681207999999998 rpy=-3.141592653589793 -1.5707963267948966 0
- joint ak60-6v1-1-v1_회전-1: axis -0.990014 -0.12427100000000012 -0.066546 -> -0.9749849999999999 -0.009442999999999993 0.22207099999999996; child 구성요소11 -> Component11; origin xyz=0.0019298499999999997 -0.003603870000000001 0.02871041000000002 rpy=3.141592653589793 -1.5707963267948966 0 -> xyz=-0.006440049999999999 -0.0002738400000000008 0.02827455999999998 rpy=-3.141592653589793 -1.5707963267948966 0
- joint ak70-10-v1_1_회전-5: child 구성요소2 -> Component2
- joint ak70-10-v1_2_강체-10: child 구성요소6 -> Component6; origin xyz=-0.02878305 0.0 -0.015413110000000004 rpy=1.5707963267948968 -0.0 -1.5707963267948966 -> xyz=0.0013870900000000001 0.0 -0.03262062 rpy=1.5707963267948966 6.902532920683855e-31 -1.5707963267948966
- joint ak70-10-v1_2_회전-9: axis -7.447951350553661e-31 0.47207000000000005 -0.881561 -> 7.881485638235972e-31 0.9990969999999999 0.042483; child 구성요소5 -> Component5; origin xyz=0.005641909999999999 0.0 0.0030212099999999977 rpy=-1.5707963267948966 -0.0 -1.5707963267948966 -> xyz=-0.00027189000000000005 0.0 0.0063941300000000005 rpy=-1.5707963267948966 6.902532920683855e-31 -1.5707963267948966

Commit message: Update sfbot.urdf

File: sfbot/sfbot.urdf (robot description, URDF)
Before this commit: robot sfbot, 15 links, 14 joints
Joints:
- removed joint Component2_강체-6
- removed joint Component3_강체-7
- removed joint Component4_강체-8
- removed joint Component5_강체-11
- removed joint Component7_강체-12
- removed joint Component8_1_강체-17
- removed joint Component9_강체-16
- removed joint Component9_강체-19
- removed joint ak60-6v1-1-v1_강체-13
- removed joint ak60-6v1-1-v1_회전-1
- removed joint ak70-10-v1_1_회전-5
- removed joint ak70-10-v1_2_강체-10
- removed joint ak70-10-v1_2_회전-9
- removed joint base_link_강체-4
- added joint Component2_fix-3: type fixed, parent Component2, child Component3, origin xyz=0.02 0.0 0.0 rpy=-3.141592653589793 -1.5707963267948966 0
- added joint Component3_fix-4: type fixed, parent Component3, child Component4, origin xyz=2.218671295934097e-34 3.4124888101640537e-66 0.01800000000000001 rpy=-3.0814879110195774e-32 2.736911063134409e-48 -5.551115123125782e-17
- added joint Component4_fix-5: type fixed, parent Component4, child ak70-10-v1_2, origin xyz=0.01082865 -0.012149730000000001 0.056999999999999995 rpy=-1.5707963267948966 7.395570986446986e-32 5.5511151231257815e-17
- added joint Component5_fix-8: type fixed, parent Component5, child Component7, origin xyz=0.0 0.018663179999999998 0.01663388 rpy=1.5707963267948966 -1.5707963267948966 0
- added joint Component7_fix-9: type fixed, parent Component7, child Component8_1, origin xyz=-0.001261729999999992 -0.016958210000000005 -0.014519890000000002 rpy=7.557866748226106e-17 -6.518246424920506e-18 -5.5511151231257815e-17
- added joint Component8_1_fix-10: type fixed, parent Component8_1, child Component9, origin xyz=-0.02491717000000001 -0.07056790000000003 -0.011491559999999987 rpy=3.141592653589793 2.1919201952020058e-17 0.0
- added joint Component9_fix-11: type fixed, parent Component9, child Component8_2, origin xyz=-0.05588981000000004 0.0 -0.06270829 rpy=-1.611776653068683e-17 -6.996850281877054e-18 -5.551115123125783e-17
- added joint Component9_fix-12: type fixed, parent Component9, child ak60-6v1-1-v1, origin xyz=-0.040407410000000005 -0.0018871499999999842 -0.02024673 rpy=1.5707963267948946 -6.996850281877054e-18 -5.551115123125783e-17
- added joint ak60-6v1-1-v1_con-14: type continuous, parent ak60-6v1-1-v1, child Component11, origin xyz=-0.011477139999999775 0.010229200000000046 -0.024589409999999957 rpy=-1.1973097379898163e-16 1.5707963267948872 0, axis -0.8479109999999997 -0.35273099999999996 0.3957629999999999
- added joint ak60-6v1-1-v1_fix-13: type fixed, parent ak60-6v1-1-v1, child Component10, origin xyz=-0.01088349999999978 0.009700100000000047 -0.023317539999999966 rpy=-1.1973097379898163e-16 1.5707963267948872 0
- added joint ak70-10-v1_1_con-2: type continuous, parent ak70-10-v1_1, child Component2, origin xyz=0.0 0.0 0.03905 rpy=-3.141592653589793 -1.5707963267948966 0, axis -1.0 -4.75865530677569e-32 -0.0
- added joint ak70-10-v1_2_con-7: type continuous, parent ak70-10-v1_2, child Component5, origin xyz=0.00425821 0.0 -0.004777709999999999 rpy=-1.5707963267948966 3.8826747678846675e-31 -1.5707963267948966, axis -2.9445298249596316e-31 -0.746527 -0.665355
- added joint ak70-10-v1_2_fix-6: type fixed, parent ak70-10-v1_2, child Component6, origin xyz=-0.0217239 0.0 0.024374180000000002 rpy=1.5707963267948966 3.8826747678846675e-31 -1.5707963267948966
- added joint base_link_fix-1: type fixed, parent base_link, child ak70-10-v1_1, origin xyz=0.0 0.0 0.023 rpy=0.0 -0.0 0.0
